File: din_isolated_onion_SPI.sch (KiCad schematic (older format))
At the start: 11 parts, among them J1 Conn_01x16, J2 Conn_01x16, J3 Conn_01x10, U1 Omega2+, U2 SI8661AB-B-IS1

Commit message: Add GPIO-CS Mux pins
Parts:
- removed JP2, JP3: Jumper_NO_Small, Jumper:SolderJumper-2_P1.3mm_Open_Pad1.0x1.5mm, symbol Device:Jumper_NO_Small
- added CS1, CS2, GP19, GP2, GP20, GP5, GP6, GP7: TestPoint, TestPoint:TestPoint_THTPad_D1.0mm_Drill0.5mm, symbol Connector:TestPoint
- renumbered TP1 to FW_RST1
Connections:
- wire segments 71 -> 77
Changed lines of the file:
@@
 	5055 1845 4565 1845
 $Comp
-L Connector:TestPoint TP1
+L Connector:TestPoint FW_RST1
 U 1 1 5D151FE3
 P 4565 2045
-F 0 "TP1" V 4519 2233 50  0000 L CNN
+F 0 "FW_RST1" V 4519 2233 50  0000 L CNN
 F 1 "TestPoint" V 4610 2233 50  0000 L CNN
 F 2 "TestPoint:TestPoint_Pad_1.5x1.5mm" H 4765 2045 50  0001 C CNN
@@
 $EndComp
 Wire Wire Line
-	2235 2810 2815 2810
+	2235 2810 2745 2810
 Wire Wire Line
 	2815 2810 2815 2145
@@
 	2750 2045 2750 2710
 Wire Wire Line
-	2750 2710 2235 2710
-Wire Wire Line
-	2235 2610 2685 2610
+	2750 2710 2645 2710
+Wire Wire Line
+	2235 2610 2550 2610
 Wire Wire Line
 	2685 2610 2685 1945
@@
 	2610 1845 2610 2510
 Wire Wire Line
-	2610 2510 2235 2510
+	2610 2510 2455 2510
 Wire Wire Line
 	3165 1745 2570 1745
@@
 	2570 1745 2570 2410
 Wire Wire Line
-	2570 2410 2235 2410
+	2570 2410 2370 2410
 Wire Wire Line
 	3165 1645 2515 1645
@@
 	2515 1645 2515 2310
 Wire Wire Line
-	2515 2310 2235 2310
+	2515 2310 2295 2310
 Wire Wire Line
 	2235 3510 2415 3510
@@
 3V3_O
 $Comp
-L Device:Jumper_NO_Small JP3
-U 1 1 5D16E0D1
-P 4595 4600
-F 0 "JP3" H 4595 4415 50  0000 C CNN
-F 1 "Jumper_NO_Small" H 4595 4506 50  0000 C CNN
-F 2 "Jumper:SolderJumper-2_P1.3mm_Open_Pad1.0x1.5mm" H 4595 4600 50  0001 C CNN
-F 3 "~" H 4595 4600 50  0001 C CNN
-	1    4595 4600
-	-1   0    0    1
-$EndComp
-$Comp
-L Device:Jumper_NO_Small JP2
-U 1 1 5D16E11E
-P 4590 4435
-F 0 "JP2" H 4590 4250 50  0000 C CNN
-F 1 "Jumper_NO_Small" H 4590 4341 50  0000 C CNN
-F 2 "Jumper:SolderJumper-2_P1.3mm_Open_Pad1.0x1.5mm" H 4590 4435 50  0001 C CNN
-F 3 "~" H 4590 4435 50  0001 C CNN
-	1    4590 4435
-	-1   0    0    1
-$EndComp
+L Connector:TestPoint GP2
+U 1 1 5D16A3CD
+P 2295 2310
+F 0 "GP2" H 2237 2337 50  0000 R CNN
+F 1 "TestPoint" H 2237 2428 50  0000 R CNN
+F 2 "TestPoint:TestPoint_THTPad_D1.0mm_Drill0.5mm" H 2495 2310 50  0001 C CNN
+F 3 "~" H 2495 2310 50  0001 C CNN
+	1    2295 2310
+	-1   0    0    1
+$EndComp
+$Comp
+L Connector:TestPoint GP5
+U 1 1 5D16A4AB
+P 2370 2410
+F 0 "GP5" H 2312 2437 50  0000 R CNN
+F 1 "TestPoint" H 2312 2528 50  0000 R CNN
+F 2 "TestPoint:TestPoint_THTPad_D1.0mm_Drill0.5mm" H 2570 2410 50  0001 C CNN
+F 3 "~" H 2570 2410 50  0001 C CNN
+	1    2370 2410
+	-1   0    0    1
+$EndComp
+Connection ~ 2370 2410
+Wire Wire Line
+	2370 2410 2235 2410
+$Comp
+L Connector:TestPoint GP6
+U 1 1 5D16A4F1
+P 2455 2510
+F 0 "GP6" H 2397 2537 50  0000 R CNN
+F 1 "TestPoint" H 2397 2628 50  0000 R CNN
+F 2 "TestPoint:TestPoint_THTPad_D1.0mm_Drill0.5mm" H 2655 2510 50  0001 C CNN
+F 3 "~" H 2655 2510 50  0001 C CNN
+	1    2455 2510
+	-1   0    0    1
+$EndComp
+Connection ~ 2455 2510
+Wire Wire Line
+	2455 2510 2235 2510
+$Comp
+L Connector:TestPoint GP7
+U 1 1 5D16A525
+P 2550 2610
+F 0 "GP7" H 2492 2637 50  0000 R CNN
+F 1 "TestPoint" H 2492 2728 50  0000 R CNN
+F 2 "TestPoint:TestPoint_THTPad_D1.0mm_Drill0.5mm" H 2750 2610 50  0001 C CNN
+F 3 "~" H 2750 2610 50  0001 C CNN
+	1    2550 2610
+	-1   0    0    1
+$EndComp
+Connection ~ 2550 2610
+Wire Wire Line
+	2550 2610 2685 2610
+$Comp
+L Connector:TestPoint GP19
+U 1 1 5D16A55F
+P 2645 2710
+F 0 "GP19" H 2587 2737 50  0000 R CNN
+F 1 "TestPoint" H 2587 2828 50  0000 R CNN
+F 2 "TestPoint:TestPoint_THTPad_D1.0mm_Drill0.5mm" H 2845 2710 50  0001 C CNN
+F 3 "~" H 2845 2710 50  0001 C CNN
+	1    2645 2710
+	-1   0    0    1
+$EndComp
+Connection ~ 2645 2710
+Wire Wire Line
+	2645 2710 2235 2710
+$Comp
+L Connector:TestPoint GP20
+U 1 1 5D16A5AD
+P 2745 2810
+F 0 "GP20" H 2687 2837 50  0000 R CNN
+F 1 "TestPoint" H 2687 2928 50  0000 R CNN
+F 2 "TestPoint:TestPoint_THTPad_D1.0mm_Drill0.5mm" H 2945 2810 50  0001 C CNN
+F 3 "~" H 2945 2810 50  0001 C CNN
+	1    2745 2810
+	-1   0    0    1
+$EndComp
+Connection ~ 2745 2810
+Wire Wire Line
+	2745 2810 2815 2810
+Connection ~ 2295 2310
+Wire Wire Line
+	2295 2310 2235 2310
+$Comp
+L Connector:TestPoint CS1
+U 1 1 5D16AF39
+P 2555 4545
+F 0 "CS1" H 2497 4572 50  0000 R CNN
+F 1 "TestPoint" H 2497 4663 50  0000 R CNN
+F 2 "TestPoint:TestPoint_THTPad_D1.0mm_Drill0.5mm" H 2755 4545 50  0001 C CNN
+F 3 "~" H 2755 4545 50  0001 C CNN
+	1    2555 4545
+	-1   0    0    1
+$EndComp
+$Comp
+L Connector:TestPoint CS2
+U 1 1 5D16B155
+P 2705 4545
+F 0 "CS2" H 2647 4572 50  0000 R CNN
+F 1 "TestPoint" H 2647 4663 50  0000 R CNN
+F 2 "TestPoint:TestPoint_THTPad_D1.0mm_Drill0.5mm" H 2905 4545 50  0001 C CNN
+F 3 "~" H 2905 4545 50  0001 C CNN
+	1    2705 4545
+	-1   0    0    1
+$EndComp
+Text GLabel 2555 4545 1    50   Input ~ 0
+CS1_O
+Text GLabel 2705 4545 1    50   Input ~ 0
+CS2_O
 $EndSCHEMATC

Commit message: Add reset IC and finalize test points
Parts:
- added 3V3, DONE1, WAKE1: TestPoint, TestPoint:TestPoint_THTPad_D1.0mm_Drill0.5mm, symbol Connector:TestPoint
- added GND1: GND, TestPoint:TestPoint_THTPad_D1.0mm_Drill0.5mm, symbol Connector:TestPoint
- added LOGO1: Logo_Open_Hardware_Large, Symbol:OSHW-Logo2_7.3x6mm_SilkScreen, symbol Graphic:Logo_Open_Hardware_Large
- added R1: 29.4K, Resistor_SMD:R_0603_1608Metric, symbol Device:R
- added RST1: Jumper_2_Bridged, Jumper:SolderJumper-2_P1.3mm_Bridged_Pad1.0x1.5mm, symbol Jumper:Jumper_2_Bridged
- added U3: TPL5010-Q1, Package_TO_SOT_SMD:SOT-23-6, symbol tpl5010-q1:TPL5010-Q1
- CS1: value TestPoint -> ChipSel1
- CS2: value TestPoint -> ChipSel2
- renumbered JP1 to VCC1
Connections:
- net labels added: ~RST
Changed lines of the file:
@@
 $EndComp
 $Comp
-L Jumper:Jumper_2_Bridged JP1
+L Jumper:Jumper_2_Bridged VCC1
 U 1 1 5D16821A
 P 3860 1120
-F 0 "JP1" H 3860 1315 50  0000 C CNN
+F 0 "VCC1" H 3860 1315 50  0000 C CNN
 F 1 "Jumper_2_Bridged" H 3860 1224 50  0000 C CNN
 F 2 "Jumper:SolderJumper-2_P1.3mm_Bridged_Pad1.0x1.5mm" H 3860 1120 50  0001 C CNN
@@
 U 1 1 5D16AF39
 P 2555 4545
-F 0 "CS1" H 2497 4572 50  0000 R CNN
-F 1 "TestPoint" H 2497 4663 50  0000 R CNN
+F 0 "CS1" H 2620 4765 50  0000 R CNN
+F 1 "ChipSel1" V 2550 5140 50  0001 R CNN
 F 2 "TestPoint:TestPoint_THTPad_D1.0mm_Drill0.5mm" H 2755 4545 50  0001 C CNN
 F 3 "~" H 2755 4545 50  0001 C CNN
@@
 U 1 1 5D16B155
 P 2705 4545
-F 0 "CS2" H 2647 4572 50  0000 R CNN
-F 1 "TestPoint" H 2647 4663 50  0000 R CNN
+F 0 "CS2" H 2760 4765 50  0000 R CNN
+F 1 "ChipSel2" V 2695 5140 50  0001 R CNN
 F 2 "TestPoint:TestPoint_THTPad_D1.0mm_Drill0.5mm" H 2905 4545 50  0001 C CNN
 F 3 "~" H 2905 4545 50  0001 C CNN
@@
 Text GLabel 2705 4545 1    50   Input ~ 0
 CS2_O
+$Comp
+L tpl5010-q1:TPL5010-Q1 U3
+U 1 1 5D173C02
+P 2730 5550
+F 0 "U3" H 2730 5915 50  0000 C CNN
+F 1 "TPL5010-Q1" H 2730 5824 50  0000 C CNN
+F 2 "Package_TO_SOT_SMD:SOT-23-6" H 2780 5550 50  0001 C CNN
+F 3 "" H 2780 5550 50  0001 C CNN
+	1    2730 5550
+	1    0    0    -1
+$EndComp
+Text GLabel 2330 5450 0    50   Input ~ 0
+3V3_C
+Text GLabel 2330 5550 0    50   Input ~ 0
+GND_C
+$Comp
+L Device:R R1
+U 1 1 5D173F56
+P 2180 5650
+F 0 "R1" V 2020 5650 50  0000 C CNN
+F 1 "29.4K" V 2090 5645 50  0000 C CNN
+F 2 "Resistor_SMD:R_0603_1608Metric" V 2110 5650 50  0001 C CNN
+F 3 "~" H 2180 5650 50  0001 C CNN
+	1    2180 5650
+	0    -1   -1   0
+$EndComp
+Text GLabel 2030 5650 0    50   Input ~ 0
+GND_C
+Text GLabel 5055 1845 2    50   Input ~ 0
+~RST
+$Comp
+L Connector:TestPoint GND1
+U 1 1 5D176CB2
+P 2880 4550
+F 0 "GND1" H 2945 4765 50  0000 R CNN
+F 1 "GND" H 2945 4845 50  0001 R CNN
+F 2 "TestPoint:TestPoint_THTPad_D1.0mm_Drill0.5mm" H 3080 4550 50  0001 C CNN
+F 3 "~" H 3080 4550 50  0001 C CNN
+	1    2880 4550
+	-1   0    0    1
+$EndComp
+$Comp
+L Connector:TestPoint 3V3
+U 1 1 5D176D00
+P 3030 4555
+F 0 "3V3" H 3085 4765 50  0000 R CNN
+F 1 "TestPoint" V 3015 5155 50  0001 R CNN
+F 2 "TestPoint:TestPoint_THTPad_D1.0mm_Drill0.5mm" H 3230 4555 50  0001 C CNN
+F 3 "~" H 3230 4555 50  0001 C CNN
+	1    3030 4555
+	-1   0    0    1
+$EndComp
+Text GLabel 2880 4550 1    50   Input ~ 0
+GND_C
+Text GLabel 3030 4555 1    50   Input ~ 0
+3V3_C
+Text GLabel 3530 5450 2    50   Output ~ 0
+~RST
+$Comp
+L Connector:TestPoint WAKE1
+U 1 1 5D178EE3
+P 3130 5550
+F 0 "WAKE1" V 3130 5738 50  0000 L CNN
+F 1 "TestPoint" V 3175 5738 50  0001 L CNN
+F 2 "TestPoint:TestPoint_THTPad_D1.0mm_Drill0.5mm" H 3330 5550 50  0001 C CNN
+F 3 "~" H 3330 5550 50  0001 C CNN
+	1    3130 5550
+	0    1    1    0
+$EndComp
+$Comp
+L Connector:TestPoint DONE1
+U 1 1 5D178F5E
+P 3130 5650
+F 0 "DONE1" V 3130 5837 50  0000 L CNN
+F 1 "TestPoint" V 3175 5838 50  0001 L CNN
+F 2 "TestPoint:TestPoint_THTPad_D1.0mm_Drill0.5mm" H 3330 5650 50  0001 C CNN
+F 3 "~" H 3330 5650 50  0001 C CNN
+	1    3130 5650
+	0    1    1    0
+$EndComp
+$Comp
+L Jumper:Jumper_2_Bridged RST1
+U 1 1 5D17969E
+P 3330 5450
+F 0 "RST1" H 3330 5645 50  0000 C CNN
+F 1 "Jumper_2_Bridged" H 3330 5554 50  0000 C CNN
+F 2 "Jumper:SolderJumper-2_P1.3mm_Bridged_Pad1.0x1.5mm" H 3330 5450 50  0001 C CNN
+F 3 "~" H 3330 5450 50  0001 C CNN
+	1    3330 5450
+	1    0    0    -1
+$EndComp
+$Comp
+L Graphic:Logo_Open_Hardware_Large LOGO1
+U 1 1 5D17A97C
+P 8355 5530
+F 0 "LOGO1" H 8355 6030 50  0001 C CNN
+F 1 "Logo_Open_Hardware_Large" H 8355 5130 50  0001 C CNN
+F 2 "Symbol:OSHW-Logo2_7.3x6mm_SilkScreen" H 8355 5530 50  0001 C CNN
+F 3 "~" H 8355 5530 50  0001 C CNN
+	1    8355 5530
+	1    0    0    -1
+$EndComp
 $EndSCHEMATC

Commit message: Switch to TSOT for hardware reset
Parts:
- C1, C2: value C_Small -> 100nF
- U3: footprint Package_TO_SOT_SMD:SOT-23-6 -> Package_TO_SOT_SMD:TSOT-23-6
Changed lines of the file:
@@
 P 9730 2335
 F 0 "C1" H 9822 2381 50  0000 L CNN
-F 1 "C_Small" H 9822 2290 50  0000 L CNN
+F 1 "100nF" H 9822 2290 50  0000 L CNN
 F 2 "Capacitor_SMD:C_0603_1608Metric" H 9730 2335 50  0001 C CNN
 F 3 "~" H 9730 2335 50  0001 C CNN
@@
 P 9920 2335
 F 0 "C2" H 10012 2381 50  0000 L CNN
-F 1 "C_Small" H 10012 2290 50  0000 L CNN
+F 1 "100nF" H 10012 2290 50  0000 L CNN
 F 2 "Capacitor_SMD:C_0603_1608Metric" H 9920 2335 50  0001 C CNN
 F 3 "~" H 9920 2335 50  0001 C CNN
@@
 F 0 "U3" H 2730 5915 50  0000 C CNN
 F 1 "TPL5010-Q1" H 2730 5824 50  0000 C CNN
-F 2 "Package_TO_SOT_SMD:SOT-23-6" H 2780 5550 50  0001 C CNN
+F 2 "Package_TO_SOT_SMD:TSOT-23-6" H 2780 5550 50  0001 C CNN
 F 3 "" H 2780 5550 50  0001 C CNN
 	1    2730 5550

Commit message: Add quad buffer and GPIO LED's
Parts:
- added D1, D2, D3, D4, D5, D6: LED, LED_SMD:LED_0603_1608Metric, symbol Device:LED
- added R2, R3, R4, R5, R6, R7: 330R, Resistor_SMD:R_0603_1608Metric, symbol Device:R
- added U4: 74LVC125, Package_SO:TSSOP-14_4.4x5mm_P0.65mm, symbol 74xx:74LVC125
- RST1: value Jumper_2_Bridged -> Jumper_2_Open; footprint Jumper:SolderJumper-2_P1.3mm_Bridged_Pad1.0x1.5mm -> Jumper:SolderJumper-2_P1.3mm_Open_Pad1.0x1.5mm; symbol Jumper:Jumper_2_Bridged -> Jumper:Jumper_2_Open
- renumbered GP2 to GP11, GP7 to GP15, GP6 to GP16, GP5 to GP17, GP20 to GP18
Connections:
- net labels added: GP11, GP15, GP16, GP17, GP18, GP19, MISO_O_ISO
- wire segments 77 -> 86

Commit message: Move parts into place on PCB for route
Parts:
- removed CS1: ChipSel1, TestPoint:TestPoint_THTPad_D1.0mm_Drill0.5mm, symbol Connector:TestPoint
- removed CS2: ChipSel2, TestPoint:TestPoint_THTPad_D1.0mm_Drill0.5mm, symbol Connector:TestPoint
- added MET_SEL1: MET_S, TestPoint:TestPoint_THTPad_D1.0mm_Drill0.5mm, symbol Connector:TestPoint
- added U5: NL7SZ19, Package_TO_SOT_SMD:SOT-23-6, symbol NL7SZ19:NL7SZ19
Connections:
- net labels added: CSMUX_0, CSMUX_1, CS_SPARE
- net labels removed: CS1_O, CS2_O
Changed lines of the file:
@@
 Text GLabel 7350 2160 0    50   Input ~ 0
 MOSI_O
-Text GLabel 7350 2260 0    50   Input ~ 0
+Text GLabel 2410 6365 0    50   Input ~ 0
 CS0_O
 Text GLabel 7350 2460 0    50   Input ~ 0
-CS1_O
+CSMUX_1
 Text GLabel 7350 2560 0    50   Input ~ 0
-CS2_O
+CS_SPARE
 Text GLabel 9150 2060 2    50   Output ~ 0
 CLK_E
@@
 Wire Wire Line
 	2295 2310 2235 2310
-$Comp
-L Connector:TestPoint CS1
-U 1 1 5D16AF39
-P 2555 4545
-F 0 "CS1" H 2620 4765 50  0000 R CNN
-F 1 "ChipSel1" V 2550 5140 50  0001 R CNN
-F 2 "TestPoint:TestPoint_THTPad_D1.0mm_Drill0.5mm" H 2755 4545 50  0001 C CNN
-F 3 "~" H 2755 4545 50  0001 C CNN
-	1    2555 4545
-	-1   0    0    1
-$EndComp
-$Comp
-L Connector:TestPoint CS2
-U 1 1 5D16B155
-P 2705 4545
-F 0 "CS2" H 2760 4765 50  0000 R CNN
-F 1 "ChipSel2" V 2695 5140 50  0001 R CNN
-F 2 "TestPoint:TestPoint_THTPad_D1.0mm_Drill0.5mm" H 2905 4545 50  0001 C CNN
-F 3 "~" H 2905 4545 50  0001 C CNN
-	1    2705 4545
-	-1   0    0    1
-$EndComp
-Text GLabel 2555 4545 1    50   Input ~ 0
-CS1_O
-Text GLabel 2705 4545 1    50   Input ~ 0
-CS2_O
+Text GLabel 3010 6365 2    50   Output ~ 0
+CSMUX_0
+Text GLabel 3010 6565 2    50   Output ~ 0
+CSMUX_1
 $Comp
 L tpl5010-q1:TPL5010-Q1 U3
@@
 	5050 4920 5050 5675
 Text GLabel 5350 4460 2    50   Input ~ 0
-CS0_O
+CSMUX_0
 Text GLabel 5350 5170 2    50   Input ~ 0
-CS1_O
+CSMUX_1
 Text GLabel 5350 5925 2    50   Input ~ 0
-CS2_O
+CS_SPARE
 Text GLabel 5045 4915 0    50   Output ~ 0
 MISO_O
@@
 	1    0    0    -1
 $EndComp
+$Comp
+L NL7SZ19:NL7SZ19 U5
+U 1 1 5D5A3EC1
+P 2710 6615
+F 0 "U5" H 2710 7090 50  0000 C CNN
+F 1 "NL7SZ19" H 2710 6999 50  0000 C CNN
+F 2 "Package_TO_SOT_SMD:SOT-23-6" H 2710 6615 50  0001 C CNN
+F 3 "" H 2710 6615 50  0001 C CNN
+	1    2710 6615
+	1    0    0    -1
+$EndComp
+Text GLabel 7350 2260 0    50   Input ~ 0
+CSMUX_0
+Text GLabel 3010 6465 2    50   Input ~ 0
+3V3_C
+Text GLabel 2410 6465 0    50   Input ~ 0
+GND_C
+$Comp
+L Connector:TestPoint MET_SEL1
+U 1 1 5D5B0E57
+P 2410 6565
+F 0 "MET_SEL1" V 2405 7050 50  0000 R CNN
+F 1 "MET_S" H 2475 6860 50  0001 R CNN
+F 2 "TestPoint:TestPoint_THTPad_D1.0mm_Drill0.5mm" H 2610 6565 50  0001 C CNN
+F 3 "~" H 2610 6565 50  0001 C CNN
+	1    2410 6565
+	0    -1   -1   0
+$EndComp
 $EndSCHEMATC

Commit message: Partially complete routing
Parts:
- removed 3V3: TestPoint, TestPoint:TestPoint_THTPad_D1.0mm_Drill0.5mm, symbol Connector:TestPoint
- removed GND1: GND, TestPoint:TestPoint_THTPad_D1.0mm_Drill0.5mm, symbol Connector:TestPoint
- added C3: 100nF, Capacitor_SMD:C_0603_1608Metric, symbol Device:C_Small
- added J4: Test_Power_Bridge, Connector_PinHeader_2.54mm:PinHeader_2x02_P2.54mm_Vertical, symbol Connector_Generic:Conn_02x02_Odd_Even
Changed lines of the file:
@@
 Text GLabel 5055 1845 2    50   Input ~ 0
 ~RST
-$Comp
-L Connector:TestPoint GND1
-U 1 1 5D176CB2
-P 2880 4550
-F 0 "GND1" H 2945 4765 50  0000 R CNN
-F 1 "GND" H 2945 4845 50  0001 R CNN
-F 2 "TestPoint:TestPoint_THTPad_D1.0mm_Drill0.5mm" H 3080 4550 50  0001 C CNN
-F 3 "~" H 3080 4550 50  0001 C CNN
-	1    2880 4550
-	-1   0    0    1
-$EndComp
-$Comp
-L Connector:TestPoint 3V3
-U 1 1 5D176D00
-P 3030 4555
-F 0 "3V3" H 3085 4765 50  0000 R CNN
-F 1 "TestPoint" V 3015 5155 50  0001 R CNN
-F 2 "TestPoint:TestPoint_THTPad_D1.0mm_Drill0.5mm" H 3230 4555 50  0001 C CNN
-F 3 "~" H 3230 4555 50  0001 C CNN
-	1    3030 4555
-	-1   0    0    1
-$EndComp
-Text GLabel 2880 4550 1    50   Input ~ 0
+Text GLabel 2555 4585 0    50   Input ~ 0
 GND_C
-Text GLabel 3030 4555 1    50   Input ~ 0
+Text GLabel 2555 4685 0    50   Input ~ 0
 3V3_C
 Text GLabel 3530 5450 2    50   Output ~ 0
@@
 	0    -1   -1   0
 $EndComp
+$Comp
+L Device:C_Small C3
+U 1 1 5D5DAF0D
+P 9880 3965
+F 0 "C3" H 9972 4011 50  0000 L CNN
+F 1 "100nF" H 9972 3920 50  0000 L CNN
+F 2 "Capacitor_SMD:C_0603_1608Metric" H 9880 3965 50  0001 C CNN
+F 3 "~" H 9880 3965 50  0001 C CNN
+	1    9880 3965
+	1    0    0    -1
+$EndComp
+Text GLabel 9880 3865 1    50   Input ~ 0
+3V3_C
+$Comp
+L power:GNDD #PWR010
+U 1 1 5D5DAF15
+P 9880 4065
+F 0 "#PWR010" H 9880 3815 50  0001 C CNN
+F 1 "GNDD" H 9884 3910 50  0000 C CNN
+F 2 "" H 9880 4065 50  0001 C CNN
+F 3 "" H 9880 4065 50  0001 C CNN
+	1    9880 4065
+	1    0    0    -1
+$EndComp
+$Comp
+L Connector_Generic:Conn_02x02_Odd_Even J4
+U 1 1 5D5DFAB5
+P 2755 4585
+F 0 "J4" H 2805 4802 50  0000 C CNN
+F 1 "Test_Power_Bridge" H 2805 4711 50  0000 C CNN
+F 2 "Connector_PinHeader_2.54mm:PinHeader_2x02_P2.54mm_Vertical" H 2755 4585 50  0001 C CNN
+F 3 "~" H 2755 4585 50  0001 C CNN
+	1    2755 4585
+	1    0    0    -1
+$EndComp
+Text GLabel 3055 4585 2    50   Output ~ 0
+GND_I
+Text GLabel 3055 4685 2    50   Output ~ 0
+3V3_I
 $EndSCHEMATC
